File: hardware/StrainGaugeBoard.kicad_sch (KiCad schematic)
At the start: 33 parts, among them J10 CAN_OUT, J4 CAN_DEBUG, J5 CAN_IN

Commit message: errors fixed
Parts:
- removed R34: 10kR, symbol Device:R
- removed TP26: SPI_MISO, symbol Connector:TestPoint
- removed TP27: SPI_MOSI, symbol Connector:TestPoint
- removed TP28: SPI_SCK, symbol Connector:TestPoint
- added J6: Conn_01x06, Connector_PinHeader_2.54mm:PinHeader_1x06_P2.54mm_Vertical, symbol Connector_Generic:Conn_01x06
- F1: footprint (none) -> LHRS_Power:Fuse-3557-2; LCSC P/N (none) -> C352820; P/N (none) -> 3557-2
- JP2: footprint (none) -> Jumper:SolderJumper-2_P1.3mm_Open_RoundedPad1.0x1.5mm
- R29, R37, R40: footprint (none) -> Resistor_SMD:R_0603_1608Metric_Pad0.98x0.95mm_HandSolder; LCSC P/N (none) -> C21190; P/N (none) -> 0603WAF1001T5E
- R41, R42, R48: footprint (none) -> Resistor_SMD:R_0603_1608Metric_Pad0.98x0.95mm_HandSolder; LCSC P/N (none) -> C2930077; P/N (none) -> FRC0603F22R0TS
- R59, R60: footprint (none) -> Resistor_SMD:R_0603_1608Metric_Pad0.98x0.95mm_HandSolder; LCSC P/N (none) -> C21189; P/N (none) -> CRCW06030000Z0EE
- R64: value 16kR -> 16k; footprint (none) -> Resistor_SMD:R_0603_1608Metric_Pad0.98x0.95mm_HandSolder; P/N (none) -> 0603WAF1743T5E
- R65: value 4.7kR -> 4.7k; footprint (none) -> Resistor_SMD:R_0603_1608Metric_Pad0.98x0.95mm_HandSolder; LCSC P/N (none) -> C23162; P/N (none) -> 0603WAF4701T5E
- TP17, TP18, TP19, TP20, TP21, TP22, TP23, TP24, TP25: footprint (none) -> TestPoint:TestPoint_Loop_D1.80mm_Drill1.0mm_Beaded; symbol Connector:TestPoint -> lhrs_misc:Multimeter_TP
Connections:
- net +3.3V: now also J6.1 (Pin_1)
- net ADC_CS: now also J6.5 (Pin_5)
- net GND: now also J6.6 (Pin_6)
- net SPI_MISO: now also J6.2 (Pin_2)
- net SPI_MOSI: now also J6.3 (Pin_3)
- net SPI_SCK: now also J6.4 (Pin_4)
Other:
- removed sheet LDO 3.3V
- added sheet LDO (LDO.kicad_sch)
- note added: "Pin Header"
- moved on the sheet: D11, D17, TP17, TP18, TP19, TP20, TP21, TP22, TP23, TP24, TP25
