File: hardware/StrainGaugeBoard.kicad_sch (KiCad schematic)
At the start: 30 parts, among them J10 CAN_OUT, J4 CAN_DEBUG, J5 CAN_IN, J6 Conn_01x06

Commit message: whoops forgot to push
Parts:
- removed D11, D17: TPD2EUSB30DRTR, LHRS_ICs:TPD2EUSB30DRTR, symbol lhrs_ics:TPD2EUSB30DRTR
- removed R59: 0, Resistor_SMD:R_0603_1608Metric_Pad0.98x0.95mm_HandSolder, symbol Device:R
- added CR1: D5V0P4UR6SO-7, LHRS_ICs:D5V0P4UR6SO-7, symbol lhrs_ics:D5V0P4UR6SO-7
- F1: value Fuse -> 1A
- J4: footprint Connector_Molex:Molex_Nano-Fit_105309-xx04_1x04_P2.50mm_Vertical -> LHRS_Connectors:Molex_Nano-Fit_105309-xx04_1x04_P2.50mm_Vertical
Connections:
- net +3.3V: now also CR1.5
- net ADC_CS: now also CR1.6
- net GND: now also CR1.2
- net SPI_MISO: now also CR1.4
- net SPI_MOSI: now also CR1.3
- net SPI_SCK: now also CR1.1
- net at J10.5 (SHIELD), R60.1: now also J5.5 (SHIELD)
Other:
- sheet CAN_Transceiver ports: added 3V3; removed 3.3v
- sheet USB-C_Connector ports: added USB_D+, USB_D-; removed USB_DM, USB_DP
- note added: "Notes: I was told to use 2 1x5 connectors instead of 1 2x5. We use 2x5 for REV B"
- note removed: "I was told to use 2 1x5 connectors instead of 1 2x5. We use 2x5 for REV B"
- note removed: "Note:"
- moved on the sheet: F1, JP2, R60, R64, R65, TP25
