File: hardware/12VBuck.kicad_sch (KiCad schematic)
At the start: 14 parts, among them U3 LMR51635XDDCR

Commit message: Fixed ERC
Parts:
- U3: footprint DDC0006A-MFG -> (none)
Changed lines of the file:
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@@
 			)
 		)
-		(property "Footprint" "DDC0006A-MFG"
+		(property "Footprint" ""
 			(at 114.3 81.28 0)
 			(hide yes)

Commit message: errors fixed
Parts:
- removed TP1: V_in_12V, TestPoint:TestPoint_THTPad_D3.0mm_Drill1.5mm, symbol Connector:TestPoint
- removed TP2: CB, TestPoint:TestPoint_THTPad_D3.0mm_Drill1.5mm, symbol Connector:TestPoint
- removed TP3: FB, TestPoint:TestPoint_THTPad_D3.0mm_Drill1.5mm, symbol Connector:TestPoint
- removed TP4: SW, TestPoint:TestPoint_THTPad_D3.0mm_Drill1.5mm, symbol Connector:TestPoint
- U1: renamed from U3; footprint (none) -> LHRS_ICs:DDC0006A-MFG
- renumbered C34 to C1, C35 to C2, C36 to C3, C37 to C4, C38 to C5, C39 to C6, R20 to R1, R21 to R2
Other:
- note removed: "Test Points"

Commit message: whoops forgot to push
Parts:
- L1: footprint LHRS_Passives:74439369082 -> LHRS_Power:XAL5050822MEC; LCSC P/N (none) -> C5309356; P/N 74439369082 -> XAL5050-822MEC
- U1: LCSC P/N (none) -> C42432812; P/N (none) -> LMR51635XDDCR
Other:
- note added: "Vin: 4.6V to 60V"
Changed lines of the file:
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@@
 	(text "12V Vout"
 		(exclude_from_sim no)
-		(at 223.012 72.898 0)
+		(at 223.52 72.39 0)
+		(effects
+			(font
+				(size 1.27 1.27)
+			)
+		)
+	)
+	(text "Vin: 4.6V to 60V"
+		(exclude_from_sim no)
+		(at 74.93 85.09 0)
 		(effects
 			(font
@@
 	(text "Fsw 400khz"
 		(exclude_from_sim no)
-		(at 90.17 113.538 0)
+		(at 90.17 113.03 0)
 		(effects
 			(font
@@
 	(text "Vout 5"
 		(exclude_from_sim no)
-		(at 107.442 112.776 0)
+		(at 107.95 113.03 0)
 		(effects
 			(font
@@
 	(text "12V-5V Buck Converter"
 		(exclude_from_sim no)
-		(at 129.794 60.452 0)
+		(at 129.54 60.96 0)
 		(effects
 			(font
@@
 			)
 			(project "StrainGaugeBoard"
-				(path "/fb459b39-605b-4b65-b2c9-e248812f4f03/b92e82c5-b57f-475d-ad11-e6ea1f670827"
+				(path "/fb459b39-605b-4b65-b2c9-e248812f4f03/0369a2dd-0a30-45a9-8dbd-6310d49e6fe6"
 					(reference "#FLG05")
 					(unit 1)
@@
 			)
 			(project "StrainGaugeBoard"
-				(path "/fb459b39-605b-4b65-b2c9-e248812f4f03/b92e82c5-b57f-475d-ad11-e6ea1f670827"
+				(path "/fb459b39-605b-4b65-b2c9-e248812f4f03/0369a2dd-0a30-45a9-8dbd-6310d49e6fe6"
 					(reference "C1")
 					(unit 1)
@@
 			)
 		)
-		(property "Footprint" "LHRS_Passives:74439369082"
+		(property "Footprint" "LHRS_Power:XAL5050822MEC"
 			(at 161.29 86.36 0)
 			(hide yes)
@@
 			)
 		)
-		(property "LCSC P/N" ""
+		(property "LCSC P/N" "C5309356"
 			(at 161.29 86.36 90)
 			(hide yes)
@@
 			)
 		)
-		(property "P/N" "74439369082"
+		(property "P/N" "XAL5050-822MEC"
 			(at 161.29 86.36 90)
 			(hide yes)
@@
 			)
 			(project "StrainGaugeBoard"
-				(path "/fb459b39-605b-4b65-b2c9-e248812f4f03/b92e82c5-b57f-475d-ad11-e6ea1f670827"
+				(path "/fb459b39-605b-4b65-b2c9-e248812f4f03/0369a2dd-0a30-45a9-8dbd-6310d49e6fe6"
 					(reference "L1")
 					(unit 1)
@@
 			)
 			(project "StrainGaugeBoard"
-				(path "/fb459b39-605b-4b65-b2c9-e248812f4f03/b92e82c5-b57f-475d-ad11-e6ea1f670827"
+				(path "/fb459b39-605b-4b65-b2c9-e248812f4f03/0369a2dd-0a30-45a9-8dbd-6310d49e6fe6"
 					(reference "#FLG09")
 					(unit 1)
@@
 			)
 			(project "StrainGaugeBoard"
-				(path "/fb459b39-605b-4b65-b2c9-e248812f4f03/b92e82c5-b57f-475d-ad11-e6ea1f670827"
+				(path "/fb459b39-605b-4b65-b2c9-e248812f4f03/0369a2dd-0a30-45a9-8dbd-6310d49e6fe6"
 					(reference "#FLG03")
 					(unit 1)
@@
 			)
 			(project "StrainGaugeBoard"
-				(path "/fb459b39-605b-4b65-b2c9-e248812f4f03/b92e82c5-b57f-475d-ad11-e6ea1f670827"
+				(path "/fb459b39-605b-4b65-b2c9-e248812f4f03/0369a2dd-0a30-45a9-8dbd-6310d49e6fe6"
 					(reference "C4")
 					(unit 1)
@@
 			)
 			(project "StrainGaugeBoard"
-				(path "/fb459b39-605b-4b65-b2c9-e248812f4f03/b92e82c5-b57f-475d-ad11-e6ea1f670827"
+				(path "/fb459b39-605b-4b65-b2c9-e248812f4f03/0369a2dd-0a30-45a9-8dbd-6310d49e6fe6"
 					(reference "C6")
 					(unit 1)
@@
 			)
 			(project "StrainGaugeBoard"
-				(path "/fb459b39-605b-4b65-b2c9-e248812f4f03/b92e82c5-b57f-475d-ad11-e6ea1f670827"
+				(path "/fb459b39-605b-4b65-b2c9-e248812f4f03/0369a2dd-0a30-45a9-8dbd-6310d49e6fe6"
 					(reference "C3")
 					(unit 1)
@@
 			)
 			(project "StrainGaugeBoard"
-				(path "/fb459b39-605b-4b65-b2c9-e248812f4f03/b92e82c5-b57f-475d-ad11-e6ea1f670827"
+				(path "/fb459b39-605b-4b65-b2c9-e248812f4f03/0369a2dd-0a30-45a9-8dbd-6310d49e6fe6"
 					(reference "#FLG08")
 					(unit 1)
@@
 			)
 			(project "StrainGaugeBoard"
-				(path "/fb459b39-605b-4b65-b2c9-e248812f4f03/b92e82c5-b57f-475d-ad11-e6ea1f670827"
+				(path "/fb459b39-605b-4b65-b2c9-e248812f4f03/0369a2dd-0a30-45a9-8dbd-6310d49e6fe6"
 					(reference "R1")
 					(unit 1)
@@
 			)
 			(project "StrainGaugeBoard"
-				(path "/fb459b39-605b-4b65-b2c9-e248812f4f03/b92e82c5-b57f-475d-ad11-e6ea1f670827"
+				(path "/fb459b39-605b-4b65-b2c9-e248812f4f03/0369a2dd-0a30-45a9-8dbd-6310d49e6fe6"
 					(reference "C2")
 					(unit 1)
@@
 			)
 			(project "StrainGaugeBoard"
-				(path "/fb459b39-605b-4b65-b2c9-e248812f4f03/b92e82c5-b57f-475d-ad11-e6ea1f670827"
+				(path "/fb459b39-605b-4b65-b2c9-e248812f4f03/0369a2dd-0a30-45a9-8dbd-6310d49e6fe6"
 					(reference "R2")
 					(unit 1)
@@
 			)
 			(project "StrainGaugeBoard"
-				(path "/fb459b39-605b-4b65-b2c9-e248812f4f03/b92e82c5-b57f-475d-ad11-e6ea1f670827"
+				(path "/fb459b39-605b-4b65-b2c9-e248812f4f03/0369a2dd-0a30-45a9-8dbd-6310d49e6fe6"
 					(reference "C5")
 					(unit 1)
@@
 			)
 		)
+		(property "P/N" "LMR51635XDDCR"
+			(at 114.3 81.28 0)
+			(hide yes)
+			(show_name no)
+			(do_not_autoplace no)
+			(effects
+				(font
+					(size 1.27 1.27)
+				)
+			)
+		)
+		(property "LCSC P/N" "C42432812"
+			(at 114.3 81.28 0)
+			(hide yes)
+			(show_name no)
+			(do_not_autoplace no)
+			(effects
+				(font
+					(size 1.27 1.27)
+				)
+			)
+		)
 		(pin "4"
 		)
@@
 			)
 			(project "StrainGaugeBoard"
-				(path "/fb459b39-605b-4b65-b2c9-e248812f4f03/b92e82c5-b57f-475d-ad11-e6ea1f670827"
+				(path "/fb459b39-605b-4b65-b2c9-e248812f4f03/0369a2dd-0a30-45a9-8dbd-6310d49e6fe6"
 					(reference "U1")
 					(unit 1)
