File: hardware/48PinMCU.kicad_sch (KiCad schematic)
At the start: 35 parts, among them J3 SWD_Header, J9 SWD, SW3 Reset, SW4 SW_SPDT, U2 STM32G473CETx, Y2 Crystal

Commit message: whoops forgot to push
Parts:
- removed C71: 10u, Capacitor_SMD:C_0805_2012Metric_Pad1.18x1.45mm_HandSolder, symbol Device:C
- C16: renamed from C24; value 0.1u -> 0.1uF; Mouser Part Number MLASH168SB7104KTNA01 -> (none)
- C17: renamed from C19; value 10u -> 10uF; Mouser Part Number 08055D475KAT4A -> (none)
- C18: renamed from C37; value 0.1u -> 0.1uF; Mouser Part Number MLASH168SB7104KTNA01 -> (none)
- C19: renamed from C38; value 0.1u -> 0.1uF; Mouser Part Number MLASH168SB7104KTNA01 -> (none)
- C22: renamed from C39; value 0.1u -> 0.1uF; Mouser Part Number MLASH168SB7104KTNA01 -> (none)
- C23: renamed from C59; value 0.1u -> 0.1uF; Mouser Part Number MLASH168SB7104KTNA01 -> (none)
- C24: renamed from C63; value 1u -> 1uF; Mouser Part Number MLASH168SB7104KTNA01 -> (none)
- C25: renamed from C64; value 0.1u -> 0.1uF; Mouser Part Number MLASH168SB7104KTNA01 -> (none)
- C26: renamed from C65; value 1u -> 1uF; Mouser Part Number MLASH168SB7104KTNA01 -> (none)
- C29: renamed from C69; value 0.1u -> 0.1uF; Mouser Part Number MLASH168SB7104KTNA01 -> (none)
- C30: renamed from C73; value 0.1u -> 0.1uF; Mouser Part Number MLASH168SB7104KTNA01 -> (none)
- C31: renamed from C76; value 0.1u -> 0.1uF; Mouser Part Number MLASH168SB7104KTNA01 -> (none)
- C32: renamed from C77; value 100n -> 100nF; LCSC P/N C14663 -> C15849
- J2: renamed from J3; symbol 100PinMCU:SWD_Header_02x02 -> lhrs_connectors:SWD_Header_02x02
- R12: renamed from R57; Mouser Part Number CRCW060310K0FKEI -> (none)
- R7: renamed from R12; Mouser Part Number CRCW060310K0FKEI -> (none)
- SW1: renamed from SW3; Mouser Part Number 612-TL3365AF180QG -> (none)
- renumbered C17 to C14, C18 to C15, D7 to D4, D8 to D6, D18 to D7, FB3 to FB1, FB4 to FB2, J9 to J3, R20 to R10, R21 to R11, R58 to R14, R11 to R6, R18 to R8, R19 to R9, SW4 to SW2, Y2 to Y1
Other:
- note removed: "What do I do now thatr i have 4 channels thins kinda means 40mA all flow thorugh the ferrite bead can you explain what to do?"
