File: hardware/CAN_Transceiver.kicad_sch (KiCad schematic)
At the start: 9 parts, among them IC1 TCAN3413DR

Commit message: errors fixed
Parts:
- renumbered C16 to C20, C17 to C21, C18 to C27, C19 to C28, D4 to D5, IC1 to IC2, JP1 to JP3, R9 to R13, R10 to R17
Changed lines of the file:
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@@
 		(in_pos_files yes)
 		(dnp no)
-		(property "Reference" "C17"
+		(property "Reference" "C21"
 			(at 76.2 73.66 0)
 			(show_name no)
@@
 			)
 			(project "StrainGaugeBoard"
-				(path "/fb459b39-605b-4b65-b2c9-e248812f4f03/ed516f81-5eb5-4849-8155-19d610b15fed"
-					(reference "C17")
+				(path "/fb459b39-605b-4b65-b2c9-e248812f4f03/bec3623c-6687-4a37-ac7e-c47c7765a3b8"
+					(reference "C21")
 					(unit 1)
 				)
@@
 		(in_pos_files yes)
 		(dnp no)
-		(property "Reference" "C19"
+		(property "Reference" "C28"
 			(at 194.564 88.646 0)
 			(show_name no)
@@
 			)
 			(project "StrainGaugeBoard"
-				(path "/fb459b39-605b-4b65-b2c9-e248812f4f03/ed516f81-5eb5-4849-8155-19d610b15fed"
-					(reference "C19")
+				(path "/fb459b39-605b-4b65-b2c9-e248812f4f03/bec3623c-6687-4a37-ac7e-c47c7765a3b8"
+					(reference "C28")
 					(unit 1)
 				)
@@
 		(dnp no)
 		(fields_autoplaced yes)
-		(property "Reference" "JP1"
+		(property "Reference" "JP3"
 			(at 215.9 78.74 0)
 			(show_name no)
@@
 			)
 			(project "StrainGaugeBoard"
-				(path "/fb459b39-605b-4b65-b2c9-e248812f4f03/ed516f81-5eb5-4849-8155-19d610b15fed"
-					(reference "JP1")
+				(path "/fb459b39-605b-4b65-b2c9-e248812f4f03/bec3623c-6687-4a37-ac7e-c47c7765a3b8"
+					(reference "JP3")
 					(unit 1)
 				)
@@
 		(in_pos_files yes)
 		(dnp no)
-		(property "Reference" "C18"
+		(property "Reference" "C27"
 			(at 88.138 73.66 0)
 			(show_name no)
@@
 			)
 			(project "StrainGaugeBoard"
-				(path "/fb459b39-605b-4b65-b2c9-e248812f4f03/ed516f81-5eb5-4849-8155-19d610b15fed"
-					(reference "C18")
+				(path "/fb459b39-605b-4b65-b2c9-e248812f4f03/bec3623c-6687-4a37-ac7e-c47c7765a3b8"
+					(reference "C27")
 					(unit 1)
 				)
@@
 		(in_pos_files yes)
 		(dnp no)
-		(property "Reference" "C16"
+		(property "Reference" "C20"
 			(at 65.278 73.66 0)
 			(show_name no)
@@
 			)
 			(project "StrainGaugeBoard"
-				(path "/fb459b39-605b-4b65-b2c9-e248812f4f03/ed516f81-5eb5-4849-8155-19d610b15fed"
-					(reference "C16")
+				(path "/fb459b39-605b-4b65-b2c9-e248812f4f03/bec3623c-6687-4a37-ac7e-c47c7765a3b8"
+					(reference "C20")
 					(unit 1)
 				)
@@
 		(in_pos_files yes)
 		(dnp no)
-		(property "Reference" "R10"
+		(property "Reference" "R17"
 			(at 201.93 80.01 90)
 			(show_name no)
@@
 			)
 			(project "StrainGaugeBoard"
-				(path "/fb459b39-605b-4b65-b2c9-e248812f4f03/ed516f81-5eb5-4849-8155-19d610b15fed"
-					(reference "R10")
+				(path "/fb459b39-605b-4b65-b2c9-e248812f4f03/bec3623c-6687-4a37-ac7e-c47c7765a3b8"
+					(reference "R17")
 					(unit 1)
 				)
@@
 		(dnp no)
 		(fields_autoplaced yes)
-		(property "Reference" "D4"
+		(property "Reference" "D5"
 			(at 196.85 46.99 0)
 			(show_name no)
@@
 			)
 			(project "StrainGaugeBoard"
-				(path "/fb459b39-605b-4b65-b2c9-e248812f4f03/ed516f81-5eb5-4849-8155-19d610b15fed"
-					(reference "D4")
+				(path "/fb459b39-605b-4b65-b2c9-e248812f4f03/bec3623c-6687-4a37-ac7e-c47c7765a3b8"
+					(reference "D5")
 					(unit 1)
 				)
@@
 		(dnp no)
 		(fields_autoplaced yes)
-		(property "Reference" "IC1"
+		(property "Reference" "IC2"
 			(at 128.27 63.5 0)
 			(show_name no)
@@
 			)
 			(project "StrainGaugeBoard"
-				(path "/fb459b39-605b-4b65-b2c9-e248812f4f03/ed516f81-5eb5-4849-8155-19d610b15fed"
-					(reference "IC1")
+				(path "/fb459b39-605b-4b65-b2c9-e248812f4f03/bec3623c-6687-4a37-ac7e-c47c7765a3b8"
+					(reference "IC2")
 					(unit 1)
 				)
@@
 		(in_pos_files yes)
 		(dnp no)
-		(property "Reference" "R9"
+		(property "Reference" "R13"
 			(at 176.53 80.01 90)
 			(show_name no)
@@
 			)
 			(project "StrainGaugeBoard"
-				(path "/fb459b39-605b-4b65-b2c9-e248812f4f03/ed516f81-5eb5-4849-8155-19d610b15fed"
-					(reference "R9")
-					(unit 1)
-				)
+				(path "/fb459b39-605b-4b65-b2c9-e248812f4f03/bec3623c-6687-4a37-ac7e-c47c7765a3b8"
+					(reference "R13")
+					(unit 1)
+				)

Commit message: whoops forgot to push
Parts:
- C28: symbol ECE319K:C -> Device:C
- D5: symbol CDSOT23-T24CAN:CDSOT23-T24CAN -> lhrs_misc:CDSOT23-T24CAN; Height 1.17 -> (none); Manufacturer_Name Bourns -> (none); Mouser Part Number 652-CDSOT23-T24CAN -> (none); Mouser Price/Stock https://www.mouser.co.uk/ProductDetail/Bourns/CDSOT23-T24CA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 -> (none)
- IC1: renamed from IC2; symbol TCAN3413DR:TCAN3413DR -> lhrs_ics:TCAN3413DR
- renumbered JP3 to JP1, R17 to R15
Connections:
- net 3.3v renamed 3V3
Changed lines of the file:
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@@
 		)
 	)
-	(hierarchical_label "3.3v"
+	(hierarchical_label "3V3"
 		(shape input)
 		(at 149.86 67.31 0)
@@
 		)
 	)
-	(hierarchical_label "3.3v"
+	(hierarchical_label "3V3"
 		(shape input)
 		(at 87.63 63.5 0)
@@
 			)
 			(project "StrainGaugeBoard"
-				(path "/fb459b39-605b-4b65-b2c9-e248812f4f03/bec3623c-6687-4a37-ac7e-c47c7765a3b8"
+				(path "/fb459b39-605b-4b65-b2c9-e248812f4f03/a3e1acfa-f779-425b-b19c-81af70e27fe8"
 					(reference "C21")
 					(unit 1)
@@
 	)
 	(symbol
-		(lib_id "ECE319K:C")
+		(lib_id "Device:C")
 		(at 189.23 88.9 180)
 		(unit 1)
@@
 			)
 			(project "StrainGaugeBoard"
-				(path "/fb459b39-605b-4b65-b2c9-e248812f4f03/bec3623c-6687-4a37-ac7e-c47c7765a3b8"
+				(path "/fb459b39-605b-4b65-b2c9-e248812f4f03/a3e1acfa-f779-425b-b19c-81af70e27fe8"
 					(reference "C28")
 					(unit 1)
@@
 		(dnp no)
 		(fields_autoplaced yes)
-		(property "Reference" "JP3"
+		(property "Reference" "JP1"
 			(at 215.9 78.74 0)
 			(show_name no)
@@
 			)
 			(project "StrainGaugeBoard"
-				(path "/fb459b39-605b-4b65-b2c9-e248812f4f03/bec3623c-6687-4a37-ac7e-c47c7765a3b8"
-					(reference "JP3")
+				(path "/fb459b39-605b-4b65-b2c9-e248812f4f03/a3e1acfa-f779-425b-b19c-81af70e27fe8"
+					(reference "JP1")
 					(unit 1)
 				)
@@
 			)
 			(project "StrainGaugeBoard"
-				(path "/fb459b39-605b-4b65-b2c9-e248812f4f03/bec3623c-6687-4a37-ac7e-c47c7765a3b8"
+				(path "/fb459b39-605b-4b65-b2c9-e248812f4f03/a3e1acfa-f779-425b-b19c-81af70e27fe8"
 					(reference "C27")
 					(unit 1)
@@
 			)
 			(project "StrainGaugeBoard"
-				(path "/fb459b39-605b-4b65-b2c9-e248812f4f03/bec3623c-6687-4a37-ac7e-c47c7765a3b8"
+				(path "/fb459b39-605b-4b65-b2c9-e248812f4f03/a3e1acfa-f779-425b-b19c-81af70e27fe8"
 					(reference "C20")
 					(unit 1)
@@
 		(in_pos_files yes)
 		(dnp no)
-		(property "Reference" "R17"
+		(property "Reference" "R15"
 			(at 201.93 80.01 90)
 			(show_name no)
@@
 			)
 			(project "StrainGaugeBoard"
-				(path "/fb459b39-605b-4b65-b2c9-e248812f4f03/bec3623c-6687-4a37-ac7e-c47c7765a3b8"
-					(reference "R17")
+				(path "/fb459b39-605b-4b65-b2c9-e248812f4f03/a3e1acfa-f779-425b-b19c-81af70e27fe8"
+					(reference "R15")
 					(unit 1)
 				)
@@
 	)
 	(symbol
-		(lib_id "CDSOT23-T24CAN:CDSOT23-T24CAN")
+		(lib_id "lhrs_misc:CDSOT23-T24CAN")
 		(at 185.42 54.61 0)
 		(unit 1)
@@
 			)
 		)
-		(property "Height" "1.17"
-			(at 204.47 449.53 0)
-			(hide yes)
-			(show_name no)
-			(do_not_autoplace no)
-			(effects
-				(font
-					(size 1.27 1.27)
-				)
-				(justify left top)
-			)
-		)
-		(property "Mouser Part Number" "652-CDSOT23-T24CAN"
-			(at 204.47 549.53 0)
-			(hide yes)
-			(show_name no)
-			(do_not_autoplace no)
-			(effects
-				(font
-					(size 1.27 1.27)
-				)
-				(justify left top)
-			)
-		)
-		(property "Mouser Price/Stock" "https://www.mouser.co.uk/ProductDetail/Bourns/CDSOT23-T24CAN?qs=Z7P4xsdcg2LuAOb%2FzQ7xoQ%3D%3D"
-			(at 204.47 649.53 0)
-			(hide yes)
-			(show_name no)
-			(do_not_autoplace no)
-			(effects
-				(font
-					(size 1.27 1.27)
-				)
-				(justify left top)
-			)
-		)
-		(property "Manufacturer_Name" "Bourns"
-			(at 204.47 749.53 0)
-			(hide yes)
-			(show_name no)
-			(do_not_autoplace no)
-			(effects
-				(font
-					(size 1.27 1.27)
-				)
-				(justify left top)
-			)
-		)
 		(property "P/N" "CDSOT23-T24CAN"
 			(at 204.47 849.53 0)
@@
 			)
 			(project "StrainGaugeBoard"
-				(path "/fb459b39-605b-4b65-b2c9-e248812f4f03/bec3623c-6687-4a37-ac7e-c47c7765a3b8"
+				(path "/fb459b39-605b-4b65-b2c9-e248812f4f03/a3e1acfa-f779-425b-b19c-81af70e27fe8"
 					(reference "D5")
 					(unit 1)
@@
 	)
 	(symbol
-		(lib_id "TCAN3413DR:TCAN3413DR")
+		(lib_id "lhrs_ics:TCAN3413DR")
 		(at 111.76 71.12 0)
 		(unit 1)
@@
 		(dnp no)
 		(fields_autoplaced yes)
-		(property "Reference" "IC2"
+		(property "Reference" "IC1"
 			(at 128.27 63.5 0)
 			(show_name no)
@@
 			)
 		)
+		(property "P/N" "TCAN3413DR"
+			(at 140.97 866.04 0)
+			(hide yes)
+			(show_name no)
+			(do_not_autoplace no)
+			(effects
+				(font
+					(size 1.27 1.27)
+				)
+				(justify left top)
+			)
+		)
+		(property "LCSC P/N" "C22433320"
+			(at 111.76 71.12 0)
+			(hide yes)
+			(show_name no)
+			(do_not_autoplace no)
+			(effects
+				(font
+					(size 1.27 1.27)
+				)
+			)
+		)
 		(property "Height" "1.75"
 			(at 140.97 466.04 0)
@@
 				)
 				(justify left top)
-			)
-		)
-		(property "P/N" "TCAN3413DR"
-			(at 140.97 866.04 0)
-			(hide yes)
-			(show_name no)
-			(do_not_autoplace no)
-			(effects
-				(font
-					(size 1.27 1.27)
-				)
-				(justify left top)
-			)
-		)
-		(property "LCSC P/N" "C22433320"
-			(at 111.76 71.12 0)
-			(hide yes)
-			(show_name no)
-			(do_not_autoplace no)
-			(effects
-				(font
-					(size 1.27 1.27)
-				)
 			)
 		)
@@
 			)
 			(project "StrainGaugeBoard"
-				(path "/fb459b39-605b-4b65-b2c9-e248812f4f03/bec3623c-6687-4a37-ac7e-c47c7765a3b8"
-					(reference "IC2")
+				(path "/fb459b39-605b-4b65-b2c9-e248812f4f03/a3e1acfa-f779-425b-b19c-81af70e27fe8"
+					(reference "IC1")
 					(unit 1)
 				)
@@
 			)
 			(project "StrainGaugeBoard"
-				(path "/fb459b39-605b-4b65-b2c9-e248812f4f03/bec3623c-6687-4a37-ac7e-c47c7765a3b8"
+				(path "/fb459b39-605b-4b65-b2c9-e248812f4f03/a3e1acfa-f779-425b-b19c-81af70e27fe8"
 					(reference "R13")
 					(unit 1)
