File: hardware/StrainChannel.kicad_sch (KiCad schematic)
At the start: 19 parts, among them J8 Conn_02x05_Counter_Clockwise, U5 TS5A3166DBVR

Commit message: errors fixed
Parts:
- C40, C41: value 1nF -> 1n; footprint (none) -> Capacitor_SMD:C_0603_1608Metric_Pad1.08x0.95mm_HandSolder; P/N (none) -> CC0603JRNPO9BN102
- C43: value 10nF -> 10n; footprint (none) -> Capacitor_SMD:C_0603_1608Metric_Pad1.08x0.95mm_HandSolder; P/N (none) -> CC0603JRNPO9BN103
- C68: value 0.1uF -> 0.1u; footprint (none) -> Capacitor_SMD:C_0603_1608Metric_Pad1.08x0.95mm_HandSolder; LCSC P/N (none) -> C14663; P/N (none) -> MLASH168SB7104KTNA01
- D10: P/N (none) -> ESDA5V3SC5
- J8: footprint (none) -> LHRS_Connectors:Molex_Nano-Fit_105310-xx10_2x05_P2.50mm_Vertical; P/N (none) -> 105310-1110
- R22, R23: value 1kR -> 1k; footprint (none) -> Resistor_SMD:R_0603_1608Metric_Pad0.98x0.95mm_HandSolder; LCSC P/N (none) -> C21190; P/N (none) -> 0603WAF1001T5E
- R24, R25, R26, R27: value (none) -> 350; footprint (none) -> Resistor_SMD:R_0603_1608Metric_Pad0.98x0.95mm_HandSolder
- R28, R30: value 0R -> 0; footprint (none) -> Resistor_SMD:R_0603_1608Metric_Pad0.98x0.95mm_HandSolder; LCSC P/N (none) -> C21189; P/N (none) -> CRCW06030000Z0EE
- R50: value 100kR -> 100k; footprint (none) -> Resistor_SMD:R_0603_1608Metric_Pad0.98x0.95mm_HandSolder; LCSC P/N (none) -> C25803; P/N (none) -> 0603WAF1003T5E
- R54: value 174kR -> 174k; footprint (none) -> Resistor_SMD:R_0603_1608Metric_Pad0.98x0.95mm_HandSolder; P/N (none) -> 0603WAF1743T5E
- TP29, TP31: footprint (none) -> TestPoint:TestPoint_Pad_D1.5mm
- U5: P/N (none) -> TS5A3166DBVR
Other:
- note added: "Check cutoffs"
- note added: "Need a 0.1% low drift part"
- note added: "Use C0G/NP0 for all three caps"

Commit message: whoops forgot to push
Parts:
- removed J8: Conn_02x05_Counter_Clockwise, LHRS_Connectors:Molex_Nano-Fit_105310-xx10_2x05_P2.50mm_Vertical, symbol Connector_Generic:Conn_02x05_Counter_Clockwise
- removed R28, R30: 0, Resistor_SMD:R_0603_1608Metric_Pad0.98x0.95mm_HandSolder, symbol Device:R
- added J8: Gauge, Connector_Phoenix_MSTB:PhoenixContact_MSTBA_2,5_2-G_1x02_P5.00mm_Horizontal, symbol Connector_Generic:Conn_01x02
- R25, R26, R27: now fitted
Connections:
- net SIG+: now also J8.1 (Pin_1)
- net VDDA: now also J8.2 (Pin_2)
Other:
- note added: "Amplifier Explanation We don't need an amplifier because the ADC already has one built in. An amplifier is normally there to make a tiny signal big enough for the ADC to read. The ADS131M04 has an adjustable amplifier inside it (gain up to 128×), so the bridge's tiny voltage gets boosted before it's measured anyway. At that setting, the ADC's own noise is only about 0.5 µε. That's already finer t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"
- note added: "Quarter: J8 replaces R24 Fit R25, R26, R27 (R24 DNP)"
- note added: "S Bridge output per µε 1.65 µV F ADC range at gain 32 ±37.5 mV r That range in strain ±22,700 µε q Strain per ADC count 0.0027 µε (the 24 bits are far finer than you'll ever use) n ADC noise at gain 32, 1 kSPS (from TI's datasheet table) 0.77 µV rms e That noise in strain 0.47 µε rms p Worst-case jitter, peak to peak ~ 3 µε e_{N} Noise after averaging 16 samples ~ 0.12 µε"
- note added: "Shunt calibration switch (TS5A3166, one per channel) MCU drives SHUNT_CALx high -> switch closes -> 174k is placed across the bridge arm (SIG+ to GNDA). This simulates a known strain: 350 / (2.0 x (350 + 174k)) = ~1000 µε (GF = 2.0). R73 (100k) holds the switch OFF at power-up / reset. To calibrate: 1) switch OFF, record zero reading 2) SHUNT_CALx HIGH, record new reading 3) µε per count = 1000 /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"
- note added: "Why we don't need an additional amplifier"
- note removed: "Check cutoffs"
- note removed: "Populate only arms without a gauge Quarter: R25, R26, R27 Half: R25, R27 Full: None"
- moved on the sheet: TP29, TP31
