File: hardware/StrainGaugeChannel.kicad_sch (KiCad schematic)
At the start: 10 parts, among them U9 ADS131M04xPW

Commit message: errors fixed
Parts:
- C42: footprint (none) -> Capacitor_SMD:C_0603_1608Metric_Pad1.08x0.95mm_HandSolder; LCSC P/N (none) -> C107083; P/N (none) -> CC0603KRX7R9BB224
- C44: value 0.1u -> 1u; footprint (none) -> Capacitor_SMD:C_0603_1608Metric_Pad1.08x0.95mm_HandSolder; LCSC P/N (none) -> C15849; P/N (none) -> MLASU168SB5105KTNA01
- C45: value 0.1uF -> 0.1u; footprint (none) -> Capacitor_SMD:C_0603_1608Metric_Pad1.08x0.95mm_HandSolder; LCSC P/N (none) -> C14663; P/N (none) -> MLASH168SB7104KTNA01
- C46: value 1uF -> 1u; footprint (none) -> Capacitor_SMD:C_0603_1608Metric_Pad1.08x0.95mm_HandSolder; LCSC P/N (none) -> C15849; P/N (none) -> MLASU168SB5105KTNA01
- C48: footprint (none) -> Capacitor_SMD:C_0603_1608Metric_Pad1.08x0.95mm_HandSolder; LCSC P/N (none) -> C14663; P/N (none) -> MLASH168SB7104KTNA01
- R61, R62: value 10kR -> 10k; footprint (none) -> Resistor_SMD:R_0603_1608Metric_Pad0.98x0.95mm_HandSolder; LCSC P/N (none) -> C25804; P/N (none) -> 0603WAF1002T5E
- TP5, TP6: footprint (none) -> TestPoint:TestPoint_Loop_D1.80mm_Drill1.0mm_Beaded; symbol Connector:TestPoint -> lhrs_misc:Multimeter_TP
- U9: P/N (none) -> ADS131M04IPWR
Other:
- moved on the sheet: TP5

Commit message: whoops forgot to push
Other:
- sheet StrainChannel3: file StrainChannel.kicad_sch -> HalfBridgeChannel.kicad_sch
Changed lines of the file:
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@@
 			)
 		)
-		(property "Sheetfile" "StrainChannel.kicad_sch"
+		(property "Sheetfile" "HalfBridgeChannel.kicad_sch"
 			(at 106.68 74.2446 0)
 			(show_name no)
