File: hardware/USB-C_Connector.kicad_sch (KiCad schematic)
At the start: 6 parts, among them J3 USB_C_Receptacle_USB2.0_16P

Commit message: errors fixed
Parts:
- C78: renamed from C24; value 10uF -> 10u
- J12: renamed from J3; footprint LHRS_ICs:USB_C_Receptacle_GCT_USB4105-xx-A_16P_TopMnt_Horizontal -> LHRS_Connectors:USB_C_Receptacle_GCT_USB4105-xx-A_16P_TopMnt_Horizontal
- renumbered D7 to D21, D8 to D23, R11 to R63, R12 to R66
Changed lines of the file:
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@@
 		(in_pos_files yes)
 		(dnp no)
-		(property "Reference" "R11"
+		(property "Reference" "R63"
 			(at 86.106 48.26 90)
 			(show_name no)
@@
 			)
 			(project "StrainGaugeBoard"
-				(path "/fb459b39-605b-4b65-b2c9-e248812f4f03/3e1f507b-ac4b-41d9-a5aa-5ad5a924ba8f"
-					(reference "R11")
+				(path "/fb459b39-605b-4b65-b2c9-e248812f4f03/2bde2a13-4d99-4d83-8b03-39dcc097d6ac"
+					(reference "R63")
 					(unit 1)
 				)
@@
 		(in_pos_files yes)
 		(dnp no)
-		(property "Reference" "R12"
+		(property "Reference" "R66"
 			(at 93.726 48.26 90)
 			(show_name no)
@@
 			)
 			(project "StrainGaugeBoard"
-				(path "/fb459b39-605b-4b65-b2c9-e248812f4f03/3e1f507b-ac4b-41d9-a5aa-5ad5a924ba8f"
-					(reference "R12")
+				(path "/fb459b39-605b-4b65-b2c9-e248812f4f03/2bde2a13-4d99-4d83-8b03-39dcc097d6ac"
+					(reference "R66")
 					(unit 1)
 				)
@@
 		(dnp no)
 		(fields_autoplaced yes)
-		(property "Reference" "J3"
+		(property "Reference" "J12"
 			(at 35.56 22.86 0)
 			(show_name no)
@@
 			)
 		)
-		(property "Footprint" "LHRS_ICs:USB_C_Receptacle_GCT_USB4105-xx-A_16P_TopMnt_Horizontal"
+		(property "Footprint" "LHRS_Connectors:USB_C_Receptacle_GCT_USB4105-xx-A_16P_TopMnt_Horizontal"
 			(at 39.37 45.72 0)
 			(hide yes)
@@
 			)
 			(project "StrainGaugeBoard"
-				(path "/fb459b39-605b-4b65-b2c9-e248812f4f03/3e1f507b-ac4b-41d9-a5aa-5ad5a924ba8f"
-					(reference "J3")
+				(path "/fb459b39-605b-4b65-b2c9-e248812f4f03/2bde2a13-4d99-4d83-8b03-39dcc097d6ac"
+					(reference "J12")
 					(unit 1)
 				)
@@
 		(dnp no)
 		(fields_autoplaced yes)
-		(property "Reference" "#FLG01"
+		(property "Reference" "#FLG04"
 			(at 71.755 30.48 0)
 			(hide yes)
@@
 			)
 			(project "StrainGaugeBoard"
-				(path "/fb459b39-605b-4b65-b2c9-e248812f4f03/3e1f507b-ac4b-41d9-a5aa-5ad5a924ba8f"
-					(reference "#FLG01")
+				(path "/fb459b39-605b-4b65-b2c9-e248812f4f03/2bde2a13-4d99-4d83-8b03-39dcc097d6ac"
+					(reference "#FLG04")
 					(unit 1)
 				)
@@
 		(in_pos_files yes)
 		(dnp no)
-		(property "Reference" "D7"
+		(property "Reference" "D21"
 			(at 59.69 24.765 0)
 			(show_name no)
@@
 			)
 			(project "StrainGaugeBoard"
-				(path "/fb459b39-605b-4b65-b2c9-e248812f4f03/3e1f507b-ac4b-41d9-a5aa-5ad5a924ba8f"
-					(reference "D7")
+				(path "/fb459b39-605b-4b65-b2c9-e248812f4f03/2bde2a13-4d99-4d83-8b03-39dcc097d6ac"
+					(reference "D21")
 					(unit 1)
 				)
@@
 		(in_pos_files yes)
 		(dnp no)
-		(property "Reference" "C24"
+		(property "Reference" "C78"
 			(at 64.3128 37.9984 0)
 			(show_name no)
@@
 			)
 		)
-		(property "Value" "10uF"
+		(property "Value" "10u"
 			(at 64.3128 35.687 0)
 			(show_name no)
@@
 			)
 			(project "StrainGaugeBoard"
-				(path "/fb459b39-605b-4b65-b2c9-e248812f4f03/3e1f507b-ac4b-41d9-a5aa-5ad5a924ba8f"
-					(reference "C24")
+				(path "/fb459b39-605b-4b65-b2c9-e248812f4f03/2bde2a13-4d99-4d83-8b03-39dcc097d6ac"
+					(reference "C78")
 					(unit 1)
 				)
@@
 		(in_pos_files yes)
 		(dnp no)
-		(property "Reference" "D8"
+		(property "Reference" "D23"
 			(at 82.55 71.12 0)
 			(show_name no)
@@
 			)
 			(project "StrainGaugeBoard"
-				(path "/fb459b39-605b-4b65-b2c9-e248812f4f03/3e1f507b-ac4b-41d9-a5aa-5ad5a924ba8f"
-					(reference "D8")
-					(unit 1)
-				)
+				(path "/fb459b39-605b-4b65-b2c9-e248812f4f03/2bde2a13-4d99-4d83-8b03-39dcc097d6ac"
+					(reference "D23")
+					(unit 1)
+				)

Commit message: whoops forgot to push
Parts:
- removed D23: TPD2EUSB30DRTR, LHRS_ICs:TPD2EUSB30DRTR, symbol lhrs_ics:TPD2EUSB30DRTR
- added D2: SP0503BAHT, Package_TO_SOT_SMD:SOT-143, symbol lhrs_ics:SP0503BAH
- renumbered C78 to C7, D21 to D1, J12 to J1, R63 to R3, R66 to R4
Connections:
- net GND: now also D2.1 (A)
- net VBUS_IN: now also D2.4 (K)
- net USB_DM renamed USB_D-
- net USB_D-: now also D2.3 (K)
- net USB_DP renamed USB_D+
- net USB_D+: now also D2.2 (K)
Other:
- note removed: "5.5V working 7V breakdown 8V clamping"
